File: hw/conn.sch (KiCad schematic (older format))
At the start: 7 parts, among them SW1 SW_DIP_x04

Commit message: rebuild as serio/pario hat
Parts:
- removed SW1: SW_DIP_x04, Button_Switch_THT:SW_DIP_SPSTx04_Slide_9.78x12.34mm_W7.62mm_P2.54mm, symbol Switch:SW_DIP_x04
- removed XP10: SERVO, hat:SERVO4, symbol dronecode-conn:Servo-Conn4
- removed XP12, XP13: PWR-5V, Connector_JST:JST_PH_B2B-PH-K_1x02_P2.00mm_Vertical, symbol Connector_Generic:Conn_01x02
- removed XP14: BATT, hat:XT30, symbol Connector_Specialized:Screw_Terminal_01x02
- removed XP8: CFG ID, Connector_JST:JST_PH_B4B-PH-K_1x04_P2.00mm_Vertical, symbol Connector_Generic:Conn_01x04
Connections:
- net labels removed: +5V, +BATT, CFG_ID0, CFG_ID1, CFG_ID2, SERVO0, SERVO1, SERVO2, SERVO3, ~HAT_ID_WE
- wire segments 69 -> 9
