File: hw/dc-dc.sch (KiCad schematic (older format))
At the start: 8 parts

Commit message: rebuild as serio/pario hat
Parts:
- removed C15: 0.01, Capacitor_SMD:C_0603_1608Metric, symbol Device:C
- removed C16, C17: 10.0 50V, Capacitor_SMD:C_1206_3216Metric_Pad1.24x1.80mm_HandSolder, symbol Device:C
- removed C18: 0.47, Capacitor_SMD:C_1206_3216Metric_Pad1.24x1.80mm_HandSolder, symbol Device:C
- removed C19: 1000.0 uF 10 V, Capacitor_SMD:CP_Elec_10x10.5, symbol Device:CP
- removed DA2: LM2678SX-5.0/NOPB, Package_TO_SOT_SMD:TO-263-7_TabPin4, symbol hat-ic:LM2678SX
- removed L1: 12 uH SRR1208-120ML, Inductor_SMD:L_12x12mm_H8mm, symbol Device:L
- removed VD1: PDS760-13, hat:D-PowerDI-5, symbol Device:D_Schottky
Connections:
- net labels removed: +5V, +5Vhat, +BATT, CB, GND, VSW, Vbat
- wire segments 40 -> 0
- no-connect marks 1 -> 0
