File: hw/obc-drone-hat.sch (KiCad schematic (older format))
At the start: 4 parts

Commit message: rebuild as serio/pario hat
Parts:
- added BT1: CR1225-VBY2, hat:CR1225-VBY2, symbol Battery_Cell
- added C1, C6: 0.1, Capacitor_SMD:C_0603_1608Metric_Pad1.05x0.95mm_HandSolder, symbol obc-drone-hat-rescue_C-Device
- added C2, C3: 0.1uF, Capacitor_SMD:C_0603_1608Metric_Pad1.05x0.95mm_HandSolder, symbol C
- added C4, C5: 1uF, Capacitor_SMD:C_0603_1608Metric_Pad1.05x0.95mm_HandSolder, symbol C
- added C7, C8: 0.1, Capacitor_SMD:C_0603_1608Metric_Pad1.05x0.95mm_HandSolder, symbol C
- added DD1: DS3231, Package_SO:SOIC-16W_7.5x10.3mm_P1.27mm, symbol DS3231
- added DD2: MAX3109, Package_DFN_QFN:QFN-32-1EP_5x5mm_P0.5mm_EP3.45x3.45mm, symbol MAX3109
- added DD3: MCP23S17, Package_SO:SOIC-28W_7.5x17.9mm_P1.27mm, symbol MCP23S17
- added J1, J2: Conn_02x08_Top_Bottom, Connector_PinHeader_2.54mm:PinHeader_2x08_P2.54mm_Vertical, symbol Conn_02x08_Top_Bottom
- added J3, J4: DB9_Male, Connector_Dsub:DSUB-9_Male_Horizontal_P2.77x2.84mm_EdgePinOffset4.94mm_Housed_MountingHolesOffset7.48mm, symbol DB9_Male
- added JP1: CLK Source, Jumper:SolderJumper-3_P1.3mm_Open_RoundedPad1.0x1.5mm, symbol Jumper_3_Open
- added R1: 10k, Resistor_SMD:R_0603_1608Metric_Pad1.05x0.95mm_HandSolder, symbol R
- added R2: nc, Resistor_SMD:R_0603_1608Metric_Pad1.05x0.95mm_HandSolder, symbol R
- added XP1: Rpi_40PIN, hat:RaspberryPi-40Pin_P2.54mm, symbol Rpi_40PIN
- added ZQ1: ASFL1-24.000MHZ-EC-T, Crystal:Crystal_SMD_Abracon_ABM3B-4Pin_5.0x3.2mm, symbol ASFL1-oscillator
- MK1, MK2, MK3, MK4: symbol Mechanical:Mounting_Hole -> MountingHole
Connections:
- net labels added: +3.3V, +3Vbat, +5V, CE0, CE1, GND, HAT_CLK, RPI_GPCLK0, RPI_SCL, RPI_SDA, RPI_SPI0_MISO, RPI_SPI0_MOSI, RPI_SPI0_SCLK, U0_DCD, U0_DSR, U0_DTR, U0_RI, U0_RX, U0_TX, U1_DCD, U1_DSR, U1_DTR, U1_RI, U1_RX, U1_TX, U_V18, ZQ_CLK, ~HAT_RST, ~SER_IRQ_A, ~SER_IRQ_B, ~U0_CTS, ~U0_RTS, ~U1_CTS, ~U1_RTS
- wire segments 0 -> 192
- no-connect marks 0 -> 24
Other:
- note added: "NOTE: The chip has integrated reset\ncontroller and 50k pull-up Res."
- note added: "NOTE: fallback clock source\nif i can't setup Raspberry GPCLK0\n\nGPCLK0: 19.2 MHz\nZQ : 24.0 MHz"
- note added: "NOTEs:\n1. GPCLK0 mode 1 (19.2 MHz) used as clock source for other ICs\n2. RPI I2C already have 1.8k pull-up to 3v3\n3. RPI 3B can supply up to 500 mA at 3v3"
- note added: "Use RPi +3.3\nas power source"
