File: hw/rcio-mcu.sch (KiCad schematic (older format))
At the start: 27 parts

Commit message: rebuild as serio/pario hat
Parts:
- removed C1, C10, C2, C3, C4, C5, C6, C8, C9: 0.1, Capacitor_SMD:C_0603_1608Metric, symbol Device:C
- removed DA1: NCP361SN, Package_TO_SOT_SMD:SOT-23-5_HandSoldering, symbol poweric:NCP361SN
- removed DD2: STM32F030CCTx, Package_QFP:LQFP-48_7x7mm_P0.5mm, symbol MCU_ST_STM32:STM32F030CCTx
- removed DD3: NC7SZ157P6X, Package_TO_SOT_SMD:SOT-363_SC-70-6_Handsoldering, symbol hat-ic:NC7SZ157P6X
- removed HL1: WS2812B, LED_SMD:LED_WS2812B_PLCC4_5.0x5.0mm_P3.2mm, symbol LED:WS2812B
- removed R10, R11, R12, R14, R7, R9: 10k, Resistor_SMD:R_0603_1608Metric, symbol Device:R
- removed R13: 4.7k, Resistor_SMD:R_0603_1608Metric, symbol Device:R
- removed R6, R8: 47k, Resistor_SMD:R_0603_1608Metric, symbol Device:R
- removed VT3: DMG2305UX, Package_TO_SOT_SMD:SOT-23_Handsoldering, symbol hat-ic:DMG2305UX
- removed XP2: FrSky-XSR, Connector_JST:JST_GH_SM06B-GHS-TB_1x06-1MP_P1.25mm_Horizontal, symbol dronecode-conn:FrSky-XSR
- removed XP3: DC-Debug, Connector_JST:JST_GH_BM06B-GHS-TBT_1x06-1MP_P1.25mm_Vertical, symbol dronecode-conn:DC-Debug
- removed XP4: FAN, Connector:FanPinHeader_1x03_P2.54mm_Vertical, symbol Connector_Generic:Conn_01x03
- removed XP5: CPPM OUT, Connector_JST:JST_PH_B2B-PH-K_1x02_P2.00mm_Vertical, symbol Connector_Generic:Conn_01x02
Connections:
- net labels removed: +3.3V, +5V, +5VP, +5Vhat, ADC_IN0_Vbat, ADC_IN1_5V, CPPM_OUT, CPPM_SEL, FAN+, FAN_RPM, GND, HAT_CLK, RPI_SCL, RPI_SDA, RPI_SPI0_MISO, RPI_SPI0_MOSI, RPI_SPI0_SCLK, Rx_5V, Rx_CPPM, Rx_S.port, Rx_SBUS, SERVO0, SERVO1, SERVO2, SERVO3, STM_BOOT0, STM_CPPM, STM_U1_RX, STM_U1_TX, SWCLK, SWDIO, Vbat, WS_DOUT, ~FAN_PWM, ~RPI_SPI0_CE1, ~Rx_EN, ~STM_INT, ~STM_RESET
- wire segments 152 -> 0
- no-connect marks 13 -> 0
Other:
- note removed: "NOTE: For rev.1 will use same transistor as for ZVD.\nBut that limit to 5V only FANs."
- note removed: "NOTE: WS_DOUT can be implemented\non TIM17 CH1 (PB9), or USART5 (PB3).\n\nDecided to leave only USART5 because\ni implemented usart based driver prev."
- note removed: "NOTE: XSR module uses 5-pin conn.\nI decided to use 6-pin JST GH, to reduce nomenclature."
- note removed: "NOTE: may be replaced\nwith NC7SB3157P6X (analog sw)"
