File: hw/rpi.sch (KiCad schematic (older format))
At the start: 9 parts

Commit message: rebuild as serio/pario hat
Parts:
- removed DD1: CAT24C256WI-GT3, Package_SO:SO-8_5.3x6.2mm_P1.27mm, symbol hat-ic:CAT24
- removed R1: 1k, Resistor_SMD:R_0603_1608Metric, symbol Device:R
- removed R2, R3: 3.9k, Resistor_SMD:R_0603_1608Metric, symbol Device:R
- removed R4: 10k, Resistor_SMD:R_0603_1608Metric, symbol Device:R
- removed R5: 47k, Resistor_SMD:R_0603_1608Metric, symbol Device:R
- removed VT1: DMG2305UX, Package_TO_SOT_SMD:SOT-23_Handsoldering, symbol hat-ic:DMG2305UX
- removed VT2: DMMT5401, Package_TO_SOT_SMD:SOT-23-6_Handsoldering, symbol hat-ic:DMMT5401
Connections:
- net labels removed: +5V, CFG_ID0, CFG_ID1, CFG_ID2, ID_SCL, ID_SDA, RPI_RX, RPI_TX, STM_BOOT0, ZVD_B, ZVD_G, ~HAT_ID_WE, ~STM_INT, ~STM_RESET
- wire segments 94 -> 38
- no-connect marks 9 -> 19
Other:
- note added: "Use RPi +3.3\nas power source"
- note removed: "HAT ID EEPROM"
- note removed: "Use RPi +3.3\nas powe source"
- note removed: "Zero voltage drop diode circuit\nRecommended for HAT power supply"
