File: hw/uart.sch (KiCad schematic (older format))
At the start: 10 parts

Commit message: rebuild as serio/pario hat
Parts:
- removed XP6: TELEM1, Connector_JST:JST_GH_SM06B-GHS-TB_1x06-1MP_P1.25mm_Horizontal, symbol dronecode-conn:DC-Telemetry
- removed XP7: TELEM2, Connector_JST:JST_GH_SM06B-GHS-TB_1x06-1MP_P1.25mm_Horizontal, symbol dronecode-conn:DC-Telemetry
- added BT? (x2): CR1225-VBY2, hat:CR1225-VBY2, symbol obc-drone-hat-rescue:Battery_Cell-Device
- added C? (x2): 0.1, Capacitor_SMD:C_0603_1608Metric, symbol obc-drone-hat-rescue:C-Device
- added DD? (x2): DS3231, Package_SO:SOIC-16W_7.5x10.3mm_P1.27mm, symbol hat-ic:DS3231
- C1: renamed from C12; symbol Device:C -> obc-drone-hat-rescue:C-Device
- C2: renamed from C11; symbol Device:C -> obc-drone-hat-rescue:C-Device
- C3: renamed from C13; symbol Device:C -> obc-drone-hat-rescue:C-Device
- JP1: value Jumper_3_Open -> Jumper_1_Open; symbol Jumper:Jumper_3_Open -> obc-drone-hat-rescue:Jumper_3_Open-Jumper
- R1: renamed from R16; symbol Device:R -> obc-drone-hat-rescue:R-Device
- R2: renamed from R15; symbol Device:R -> obc-drone-hat-rescue:R-Device
- renumbered DD4 to DD1
Connections:
- net labels added: +3Vbat, RPI_SCL, RPI_SDA
- net labels removed: +5V
- wire segments 74 -> 78
- no-connect marks 9 -> 3
Other:
- note added: "NOTE: That chip has integrated reset controller and 50k pull-up R."
- moved on the sheet: C1, C2, C3, DD1, JP1, R1, R2, ZQ1
