File: hw-v2/raspi-serial-hat.sch (KiCad schematic (older format))
At the start: 41 parts, among them J1 Conn_02x10_Odd_Even, J2 DB9_Male, J3 DB9_Male, U1 DS3231, U2 MAX3109, U3 MCP23S17, U4 LT1137ACSW

Commit message: board v2, using IDC cables and with config rom.
Parts:
- removed D1, D2: LED, Diode_SMD:D_0603_1608Metric, symbol Device:LED
- removed J1: Conn_02x10_Odd_Even, Connector_PinHeader_2.54mm:PinHeader_2x10_P2.54mm_Vertical, symbol Connector_Generic:Conn_02x10_Odd_Even
- removed J2, J3: DB9_Male, Connector_Dsub:DSUB-9_Male_Vertical_P2.77x2.84mm_MountingHoles, symbol Connector1:DB9_Male
- removed JP1: CLK Source, Jumper:SolderJumper-3_P1.3mm_Open_RoundedPad1.0x1.5mm, symbol Jumper:Jumper_3_Open
- removed JP2: LED1 Enable, Jumper:SolderJumper-2_P1.3mm_Open_RoundedPad1.0x1.5mm, symbol Jumper:Jumper_2_Open
- removed JP3: LED2 Enable, Jumper:SolderJumper-2_P1.3mm_Open_RoundedPad1.0x1.5mm, symbol Jumper:Jumper_2_Open
- removed U3: MCP23S17, Package_SO:SOIC-28W_7.5x17.9mm_P1.27mm, symbol hat-ic:MCP23S17
- removed U4: LT1137ACSW, Package_SO:SOIC-28W_7.5x17.9mm_P1.27mm, symbol uarts:LT1137ACSW
- added C14, C15, C16, C26, C27: 100nF, Capacitor_SMD:C_0603_1608Metric_Pad1.05x0.95mm_HandSolder, symbol Device:C
- added C17: 100uF, Capacitor_Tantalum_SMD:CP_EIA-3528-12_Kemet-T_Pad1.50x2.35mm_HandSolder, symbol Device:CP
- added C18, C19, C20, C21, C22, C23, C24, C25: 100pF, Capacitor_SMD:C_0603_1608Metric_Pad1.05x0.95mm_HandSolder, symbol Device:C
- added J1: Conn_02x07, Connector_PinHeader_2.54mm:PinHeader_2x07_P2.54mm_Vertical, symbol Connector_Generic:Conn_02x07_Odd_Even
- added J2, J3: Conn_02x05_Odd_Even, Connector_IDC:IDC-Header_2x05_P2.54mm_Vertical, symbol Connector_Generic:Conn_02x05_Odd_Even
- added J4: Conn_02x04, Connector_PinHeader_2.54mm:PinHeader_2x04_P2.54mm_Vertical, symbol Connector_Generic:Conn_02x04_Odd_Even
- added J5, J6, J7: Conn_01x02, Connector_PinHeader_1.27mm:PinHeader_1x02_P1.27mm_Vertical, symbol Connector_Generic:Conn_01x02
- added J8: Conn_01x03, Connector_PinHeader_1.27mm:PinHeader_1x03_P1.27mm_Vertical, symbol Connector_Generic:Conn_01x03
- added MK5, MK6: MountingHole, hat:M2.5_Mounting_Hole, symbol Mechanical:MountingHole
- added R10: 10K, Resistor_SMD:R_0603_1608Metric_Pad1.05x0.95mm_HandSolder, symbol Device:R
- added R5, R6, R8, R9: 3.9K, Resistor_SMD:R_0603_1608Metric_Pad1.05x0.95mm_HandSolder, symbol Device:R
- added R7: 1K, Resistor_SMD:R_0603_1608Metric_Pad1.05x0.95mm_HandSolder, symbol Device:R
- added TP6: TestPoint, TestPoint:TestPoint_Pad_1.0x1.0mm, symbol Connector:TestPoint
- added U3: MCP23S17_SS, Package_SO:SSOP-28_5.3x10.2mm_P0.65mm, symbol Interface_Expansion:MCP23S17_SS
- added U4, U5: LT1137ACG, Package_SO:SSOP-28_5.3x10.2mm_P0.65mm, symbol uarts:LT1137ACG
- added U6: MCP23009-ESS, Package_SO:SSOP-20_5.3x7.2mm_P0.65mm, symbol hat-ic:MCP23009-ESS
- added U7: CAT24C64, Package_SO:SOIC-8_3.9x4.9mm_P1.27mm, symbol hat-ic:CAT24
- BT1: value CR1225 -> Battery_Cell; Cost/item (none) -> 0.221; Manuf Part No (none) -> BAT-HLD-012-SMT; Manufacturer (none) -> Linx Technologies; Stock Number (none) -> 712-BAT-HLD-012-SMT; Supplier (none) -> Mouser
- C1, C10, C8, C9: Cost/item (none) -> 0.084; Manuf Part No (none) -> C0603C104K4RECTU; Manufacturer (none) -> KEMET; Stock Number (none) -> 80-C0603C104K4RECTU; Supplier (none) -> Mouser
- C11, C12: value 0.1uF -> 100nF; Cost/item (none) -> 0.084; Manuf Part No (none) -> C0603C104K4RECTU; Manufacturer (none) -> KEMET; Stock Number (none) -> 80-C0603C104K4RECTU; Supplier (none) -> Mouser
- C13, C6: value 10uF Ceramic -> 10uF; Cost/item (none) -> 0.30; Manuf Part No (none) -> VJ0805G106KXYTW1BC; Manufacturer (none) -> Vishay / Vitramon; Stock Number (none) -> 77-VJ805G106KXYTW1BC; Supplier (none) -> Mouser
- C2, C4, C5: value 1uF -> 100nF; Cost/item (none) -> 0.084; Manuf Part No (none) -> C0603C104K4RECTU; Manufacturer (none) -> KEMET; Stock Number (none) -> 80-C0603C104K4RECTU; Supplier (none) -> Mouser
- C3: value 470nF -> 100nF; Cost/item (none) -> 0.084; Manuf Part No (none) -> C0603C104K4RECTU; Manufacturer (none) -> KEMET; Stock Number (none) -> 80-C0603C104K4RECTU; Supplier (none) -> Mouser
- C7: value 100uF Tant -> 100uF; symbol Device:C -> Device:CP; Cost/item (none) -> 1.14; Stock Number (none) -> 80-T520B107M10ATE070; Supplier (none) -> Mouser
- MK1, MK2, MK3, MK4: value Mounting_Hole -> MountingHole
- R1: value 10k -> 10K; Cost/item (none) -> 0.076; Manuf Part No (none) -> CRCW060310K0JNEAC; Manufacturer (none) -> Vishay; Stock Number (none) -> 71-CRCW060310K0JNEAC; Supplier (none) -> Mouser
- R2: value nc -> NO; Manuf Part No (none) -> DNF
- R3, R4: value 470 -> 10K; Cost/item (none) -> 0.076; Manuf Part No (none) -> CRCW060310K0JNEAC; Manufacturer (none) -> Vishay; Stock Number (none) -> 71-CRCW060310K0JNEAC; Supplier (none) -> Mouser
- U1: Cost/item (none) -> 6.00; Manuf Part No (none) -> DS3231S#T&R; Manufacturer (none) -> Maxim Integrated; Stock Number (none) -> 700-DS3231S#T&R-; Supplier (none) -> Mouser
- U2: Cost/item (none) -> 5.21; Manuf Part No (none) -> MAX3109ETJ+; Manufacturer (none) -> Maxim Integrated; Stock Number (none) -> 700-MAX3109ETJ+; Supplier (none) -> Mouser
- XP1: Cost/item (none) -> 1.49; Manuf Part No (none) -> 1112; Manufacturer (none) -> Adafruit; Stock Number (none) -> 485-1112; Supplier (none) -> Mouser
- ZQ1: value ASFL1-24.000MHZ-EC-T -> ASFL1-oscillator; Cost/item (none) -> 0.944; Manuf Part No (none) -> ASFL1-24.000MHZ-EC-T; Manufacturer (none) -> ABRACON; Stock Number (none) -> 815-ASFL1-24.0-EC-T; Supplier (none) -> Mouser
Connections:
- net +3V3: now also R3.2, U1.2 (Vcc), C16.1, C17.1, J1.14 (Pin_14), R10.2, R5.2, R6.2, R7.2, R8.2, R9.2, U3.9 (VDD), U6.1 (Vdd), U7.8 (Vcc); no longer U1.14 (Vbat)
- net +3Vbat: now also U1.14 (Vbat)
- net +5V: now also C26.1, C27.1, U4.13 (ON/~OFF), U4.2 (VCC), U5.13 (ON/~OFF), U5.2 (VCC)
- net CE1: now also U3.11 (~CS~)
- net GND: now also R4.1, U1.10 (GND), U1.11 (GND), U1.12 (GND), U1.13 (GND), U1.5 (GND), U1.6 (GND), U1.7 (GND), U1.8 (GND), U1.9 (GND), C16.2, C17.2, C18.1, C19.1, C20.1, C21.1, C22.1, C23.1, C24.1, C25.1, C26.2, C27.2, J1.13 (Pin_13), J2.5 (Pin_5), J3.5 (Pin_5), J5.2 (Pin_2), U3.10 (VSS), U3.15 (A0), U3.16 (A1), U3.17 (A2), U4.17 (GND), U5.17 (GND), U6.20 (GND), U6.7 (INT), U7.1 (A0), U7.2 (A1), U7.3 (A2), U7.4 (Vss); no longer R3.2, R4.2
- net HAT_CLK: now also J8.2 (Pin_2)
- net RPI_GPCLK0: now also J8.1 (Pin_1)
- net RPI_SCL: now also J6.2 (Pin_2), R8.1, U6.3 (SCL); no longer U1.16 (SCL)
- net RPI_SDA: now also J7.2 (Pin_2), R9.1, U6.4 (SDA); no longer U1.15 (SDA)
- net U0_RX: now also U4.24 (R1OUT); no longer TP4.1
- net U0_TX: now also U4.25 (T1IN); no longer TP3.1
- net U1_RX: now also U5.24 (R1OUT)
- net U1_TX: now also U5.25 (T1IN)
- net ZQ_CLK: now also J8.3 (Pin_3)
- net ~HAT_RST: now also U3.18 (~RESET~), U6.6 (~RESET)
- net ~U0_CTS: now also U4.22 (R2OUT)
- net ~U0_DCD: now also U4.21 (R3OUT)
- net ~U0_DSR: now also U4.20 (R4OUT)
- net ~U0_DTR: now also U4.19 (T3IN)
- net ~U0_RI: now also U4.18 (R5OUT)
- net ~U0_RTS: now also U4.23 (T2IN)
- net ~U1_CTS: now also U5.22 (R2OUT)
- net ~U1_DCD: now also U5.21 (R3OUT)
- net ~U1_DSR: now also U5.20 (R4OUT)
- net ~U1_DTR: now also U5.19 (T3IN)
- net ~U1_RI: now also U5.18 (R5OUT)
- net ~U1_RTS: now also U5.23 (T2IN)
- net at U1.1 (32kHz): now also TP6.1
- net CLK_INT_SW: now reaches U1.3 (~INT~/SQW)
- net CLK_INT_SW: now also U6.16 (GPB6)
- net ~SER_IRQ_B: now reaches XP1.13 (BCM27)
- net ~SER_IRQ_B: now also R10.1, U3.19 (INTB), U3.20 (INTA)
- net ID_SD: now reaches XP1.27 (BCM0_ID_SD)
- net ID_SD: now also R5.1, U7.5 (SDA)
- net ID_SC: now reaches XP1.28 (BCM1_ID_SC)
- net ID_SC: now also R6.1, U7.6 (SCL)
- net at C12.1: now also U5.3 (C1+)
- net at C12.2: now also U5.4 (C1-)
- net at C11.1: now also U4.3 (C1+)
- net at C11.2: now also U4.4 (C1-)
- net at R3.1: now also R4.2, U6.5 (ADDR)
- net RPI_SPI0_MISO renamed MISO
- net MISO: now also U3.14 (SO)
- net RPI_SPI0_MOSI renamed MOSI
- net MOSI: now also U3.13 (SI)
- net RPI_SPI0_SCLK renamed SCLK
- net SCLK: now also U3.12 (SCK)
- net V+ renamed V0+
- net V0+: now also U4.1 (V+)
- net V- renamed V1+
- net V1+: now also U5.1 (V+)
- new net: J7.1 (Pin_1), U1.15 (SDA)
- new net: J6.1 (Pin_1), U1.16 (SCL)
- new net: C14.1, U4.27 (C2-)
- new net: C14.2, U4.26 (C2+)
- new net: C15.1, U5.27 (C2-)
- new net: C15.2, U5.26 (C2+)
- new net: J5.1 (Pin_1), R7.1, U7.7 (WP)
- new net E0_RX: C20.2, J2.2 (Pin_2), U4.6 (R1IN)
- new net E0_TX: C18.2, J2.3 (Pin_3), U4.5 (T1OUT)
- new net E1_RX: C21.2, J3.2 (Pin_2), U5.6 (R1IN)
- new net E1_TX: C19.2, J3.3 (Pin_3), U5.5 (T1OUT)
- new net PA0: J4.1 (Pin_1), U3.21 (GPA0)
- new net PA1: J4.2 (Pin_2), U3.22 (GPA1)
- new net PA2: J4.3 (Pin_3), U3.23 (GPA2)
- new net PA3: J4.4 (Pin_4), U3.24 (GPA3)
- new net PA4: J4.5 (Pin_5), U3.25 (GPA4)
- new net PA5: J4.6 (Pin_6), U3.26 (GPA5)
- new net PA6: J4.7 (Pin_7), U3.27 (GPA6)
- new net PA7: J4.8 (Pin_8), U3.28 (GPA7)
- new net PB0: J1.1 (Pin_1), U3.1 (GPB0)
- new net PB1: J1.2 (Pin_2), U3.2 (GPB1)
- new net PB2: J1.3 (Pin_3), U3.3 (GPB2)
- new net PB3: J1.4 (Pin_4), U3.4 (GPB3)
- new net PB4: J1.5 (Pin_5), U3.5 (GPB4)
- new net PB5: J1.6 (Pin_6), U3.6 (GPB5)
- new net PB6: J1.7 (Pin_7), U3.7 (GPB6)
- new net PB7: J1.8 (Pin_8), U3.8 (GPB7)
- new net PC0: J1.9 (Pin_9), U6.8 (GPB0)
- new net PC1: J1.10 (Pin_10), U6.9 (GPB1)
- new net PC2: J1.11 (Pin_11), U6.12 (GPB2)
- new net PC3: J1.12 (Pin_12), U6.13 (GPB3)
- new net PC7: U6.17 (GPB7)
- new net U0_DISABLE: U4.16 (DRIVER_DISABLE), U6.14 (GPB4)
- new net U1_DISABLE: U5.16 (DRIVER_DISABLE), U6.15 (GPB5)
- new net V0-: TP3.1, U4.28 (V-)
- new net V1-: TP4.1, U5.28 (V-)
- new net ~E0_CTS: C24.2, J2.8 (Pin_8), U4.8 (R2IN)
- new net ~E0_DCD: J2.1 (Pin_1), U4.9 (R3IN)
- new net ~E0_DSR: J2.6 (Pin_6), U4.10 (R4IN)
- new net ~E0_DTR: J2.4 (Pin_4), U4.11 (T3OUT)
- new net ~E0_RI: J2.9 (Pin_9), U4.12 (R5IN)
- new net ~E0_RTS: C22.2, J2.7 (Pin_7), U4.7 (T2OUT)
- new net ~E1_CTS: C25.2, J3.8 (Pin_8), U5.8 (R2IN)
- new net ~E1_DCD: J3.1 (Pin_1), U5.9 (R3IN)
- new net ~E1_DSR: J3.6 (Pin_6), U5.10 (R4IN)
- new net ~E1_DTR: J3.4 (Pin_4), U5.11 (T3OUT)
- new net ~E1_RI: J3.9 (Pin_9), U5.12 (R5IN)
- new net ~E1_RTS: C23.2, J3.7 (Pin_7), U5.7 (T2OUT)
- no-connect marks 22 -> 19
Other:
- note added: "1:8 pot.div.\n(address)"
- note added: "8bit IO port"
- note added: "COM1"
- note added: "COM2"
- note added: "Caps: EMI smoothing"
- note added: "DS3231 has integrated reset controller and 50k pull-up Res."
- note added: "Decoupling caps"
- note added: "Dual 8bit IO port"
- note added: "Dual UART"
- note added: "GPIO"
- note added: "HAT ID"
- note added: "I2C pullup"
- note added: "IRQ (INT) on MCP23009 is grounded."
- note added: "IRQ (INTA/INTB) on MCP23S17 must be configured active-low."
- note added: "IRQ pullup"
- note added: "RPI Connector"
- note added: "RTC"
- note added: "TP: COM1 12V"
- note added: "TP: COM2 12V"
- note added: "UART CLOCK"
- note added: "ZQ is fallback clock:\n- GPCLK0: 19.2 MHz\n- ZQ : 24.0 MHz"
- note removed: "DB9 connectors:\nFCT Group: THT082016.pdf\n - THT con male (horizontal, board\n edge), height 5.5mm, width\n o/a 31.5mm, depth 13mm;\nMfr. Part No. 173109-0061\nMouser Part No 152-FHT09P5G1\n\n - THT con male (vertical) height\n 10mm to face (+6mm), width\n o/a 31.4mm, depth 12.5mm.\nMfr. Part No. 172704-0074\nMouser Part No 152-F09P-1G1\n\n\nor: \ncon male (horizontal, board\nNorComp 191-009-123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"
- note removed: "NOTE: The chip has integrated reset\ncontroller and 50k pull-up Res."
- note removed: "NOTE: fallback clock source\nIf Raspberry GPCLK0 not useful.\n\nGPCLK0: 19.2 MHz\nZQ : 24.0 MHz"
- moved on the sheet: BT1, C1, C10, C13, C2, C3, C4, C5, C6, C8, C9, MK1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
