File: hw-v3/raspi-serial-hat.sch (KiCad schematic (older format))
At the start: 75 parts, among them J1 Conn_02x07, J10 Conn_02x02, J2 Conn_02x05_Odd_Even, J3 Conn_02x05_Odd_Even, J4 Conn_02x05_Odd_Even, J5 Conn_01x02, J6 Conn_02x02, J7 Conn_01x02, J8 Conn_01x03, J9 Conn_01x02, U1 DS3231, U2 MAX3109, U3 MCP23S17_SS, U4 LT1137ACG, U5 LT1137ACG, U6 MCP23009-ESS, U7 CAT24C64

Commit message: Create gerbers and relabel schematic
Parts:
- LED1: Manuf Part No (none) -> APT1608QGW; Manufacturer (none) -> Kingbright; Stock Number (none) -> 604APT1608QGW; Supplier (none) -> Mouser
- renumbered C17 to C1, C13 to C10, C9 to C11, C10 to C12, C11 to C13, C12 to C14, C26 to C15, C27 to C16, C1 to C17, C14 to C18, C22 to C19, C4 to C2, C15 to C20, C23 to C21, C18 to C22, C19 to C23, C20 to C26, C21 to C27, C16 to C3, C5 to C4, C2 to C5, C3 to C7, C7 to C9, J7 to J1, J3 to J10, J10 to J2, J5 to J3, J9 to J4, J6 to J5, J1 to J6, J4 to J7, J2 to J9, R8 to R1, R13 to R11, R15 to R12, R16 to R13, R17 to R14, R9 to R2, R5 to R3, R6 to R4, R11 to R5, R7 to R6, R1 to R7, R3 to R8, R4 to R9, TP6 to TP1, TP7 to TP2, TP8 to TP3, TP1 to TP4, TP2 to TP5, TP3 to TP6, TP4 to TP7, U7 to U1, U1 to U2, U2 to U3, U3 to U4, U6 to U5, U4 to U6, U5 to U7
